File: HW/V1/Board/Board.kicad_pcb (KiCad board)
At the start: 2 copper layers, 99.7 x 70.1 mm, 23 parts, among them J1 Barrel_Jack, J2 +/-24V, J3 Lamp, J4 ToScanner, J5 i2cLCD, J6 toScale, Q1 IRF7341, U1 V7805-1000, U2 74HC14, U3 HX711_Module

Commit message: Done
Parts:
- removed ROT1: ROTARY-ENCODER-Ebay, Libs:ROTARY-ENCODER-Ebay
- added D1: D_Schottky, Diode_SMD:D_SMB_Handsoldering, B.Cu at (168.5, 88.5)
- added H1: MountingHole, MountingHole:MountingHole_3.2mm_M3_DIN965, F.Cu at (125.6, 54.3)
- added H2: MountingHole, MountingHole:MountingHole_3.2mm_M3_DIN965, F.Cu at (169.9, 39.7)
- added H3: MountingHole, MountingHole:MountingHole_3.2mm_M3_DIN965, F.Cu at (160.1, 78.0)
- added H4: MountingHole, MountingHole:MountingHole_3.2mm_M3_DIN965, F.Cu at (92.5, 72.6)
- added Q2: BSS138, Package_TO_SOT_SMD:SOT-23, B.Cu at (120.4, 66.6)
- added Q3: BSS138, Package_TO_SOT_SMD:SOT-23, B.Cu at (114.0, 66.6)
- added Q4: IRF7306TRPBF, Package_SO:SO-8_5.3x6.2mm_P1.27mm, B.Cu at (95.5, 49.4)
- added Q5: BSS138, Package_TO_SOT_SMD:SOT-23, B.Cu at (108.1, 66.6)
- added Q6: BSS138, Package_TO_SOT_SMD:SOT-23, B.Cu at (102.1, 66.4)
- added Q7: IRF7306TRPBF, Package_SO:SO-8_5.3x6.2mm_P1.27mm, B.Cu at (95.6, 59.4)
- added Q8: BSS138, Package_TO_SOT_SMD:SOT-23, B.Cu at (96.3, 66.3)
- added R3: 10K, Resistor_SMD:R_0805_2012Metric_Pad1.15x1.40mm_HandSolder, B.Cu at (110.9, 44.7)
- added R4: 10K, Resistor_SMD:R_0805_2012Metric_Pad1.15x1.40mm_HandSolder, B.Cu at (110.9, 47.4)
- added R5: 10K, Resistor_SMD:R_0805_2012Metric_Pad1.15x1.40mm_HandSolder, B.Cu at (91.9, 65.3)
- added R6: 10K, Resistor_SMD:R_0805_2012Metric_Pad1.15x1.40mm_HandSolder, B.Cu at (81.8, 101.3)
- added R7: 10K, Resistor_SMD:R_0805_2012Metric_Pad1.15x1.40mm_HandSolder, B.Cu at (81.9, 98.7)
- added REF**: R_Axial_DIN0207_L6.3mm_D2.5mm_P15.24mm_Horizontal, Resistor_THT:R_Axial_DIN0207_L6.3mm_D2.5mm_P15.24mm_Horizontal, F.Cu at (99.3, 93.3)
- added REF**: R_Axial_DIN0207_L6.3mm_D2.5mm_P15.24mm_Horizontal, Resistor_THT:R_Axial_DIN0207_L6.3mm_D2.5mm_P15.24mm_Horizontal, F.Cu at (95.9, 93.1)
- added REF**: R_Axial_DIN0207_L6.3mm_D2.5mm_P15.24mm_Horizontal, Resistor_THT:R_Axial_DIN0207_L6.3mm_D2.5mm_P15.24mm_Horizontal, F.Cu at (131.5, 49.5)
- added RN2: R_Network05, Resistor_THT:R_Array_SIP6, F.Cu at (106.6, 36.9)
- added RN3: R_Network05, Resistor_THT:R_Array_SIP6, F.Cu at (99.3, 72.5)
- added enc1: Rot_enc, Connector_PinSocket_2.54mm:PinSocket_1x05_P2.54mm_Vertical, F.Cu at (81.8, 82.9)
- C1, C2, C3, C4, C5, C6, C7, U2: moved to B.Cu
- J2: value +/-24V -> Screw_Terminal_01x04
- J3: value Lamp -> Screw_Terminal_01x02
- J5: footprint TerminalBlock:TerminalBlock_bornier-4_P5.08mm -> Connector_PinSocket_2.54mm:PinSocket_1x04_P2.54mm_Vertical
- Q1: value IRF7341 -> IRF7306TRPBF; footprint Package_SO:SOIC-8_3.9x4.9mm_P1.27mm -> Package_SO:SO-8_5.3x6.2mm_P1.27mm; moved to B.Cu
- R1, R2: value 10k -> 10K; moved to B.Cu
- moved C5 119.7 mm to (130.5, 46.5)
- moved Q1 100.7 mm to (95.2, 39.4), turned to 180 degrees
- moved C3 97.6 mm to (151.3, 97.4), turned to 270 degrees
- moved J3 94.0 mm to (83.4, 64.0), turned to 90 degrees
- moved C1 88.0 mm to (168.5, 82.1)
- moved R1 85.6 mm to (110.9, 39.4)
- moved R2 85.0 mm to (110.9, 42.0)
- moved C4 83.4 mm to (134.9, 97.3), turned to 180 degrees
- moved C2 81.7 mm to (133.5, 58.4)
- moved C7 76.6 mm to (105.8, 81.3), turned to 180 degrees
- moved J2 68.5 mm to (83.4, 52.2), turned to 90 degrees
- moved RN1 43.1 mm to (86.8, 84.6), turned to 90 degrees
- moved U2 32.3 mm to (98.1, 84.2), turned to 90 degrees
- moved C6 32.2 mm to (90.9, 94.7), turned to 270 degrees
- moved J6 29.5 mm to (173.8, 69.6), turned to 90 degrees
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Connections:
- A1 pad 12: LampA -> L1
- A1 pad 13: LampB -> L2
- A1 pad 14: Net-(A1-Pad14) -> L3
- A1 pad 15: Net-(A1-Pad15) -> L4
- A1 pad 16: Net-(A1-Pad16) -> Buzzer
- J2 pad 1: GND -> Net-(J2-Pad1)
- J2 pad 2: GND -> Net-(J2-Pad2)
- J2 pad 3: +24V -> Net-(J2-Pad3)
- J2 pad 4: +24V -> Net-(J2-Pad4)
- J3 pad 1: Net-(J3-Pad1) -> GND
- Q1 pad 1: GND -> +24V
- Q1 pad 2: LampA -> PullupsL1
- Q1 pad 3: GND -> +24V
- Q1 pad 4: LampB -> PullupsL2
- Q1 pad 5: Net-(J3-Pad2) -> Net-(J2-Pad3)
- Q1 pad 6: Net-(J3-Pad2) -> Net-(J2-Pad3)
- Q1 pad 7: Net-(J3-Pad1) -> Net-(J2-Pad4)
- Q1 pad 8: Net-(J3-Pad1) -> Net-(J2-Pad4)
- R1 pad 1: LampA -> PullupsL1
- R1 pad 2: GND -> Net-(Q2-Pad2)
- R2 pad 1: LampB -> PullupsL2
- R2 pad 2: GND -> Net-(Q3-Pad2)
- RN1 pad 5: SCL -> Net-(RN1-Pad5)
- RN1 pad 6: SDA -> Net-(RN1-Pad6)
Routing:
- net +24V: track 11.6 -> 159.2 mm
- net +5V: track 90.5 -> 211.3 mm
- net scannerCLK: track 24.6 -> 59.9 mm
- net Buzzer: track 0.00 -> 32.3 mm
- net GND: track 0.00 -> 31.1 mm
- net SCL: track 16.9 -> 47.4 mm
- net scaleDATA: track 52.4 -> 22.2 mm
- net BTN: track 0.00 -> 29.7 mm
- net Net-(Q2-Pad2): track 0.00 -> 29.2 mm
- net ENCB: track 0.00 -> 28.6 mm
- net ENCA: track 0.00 -> 27.3 mm
- net Net-(Q3-Pad2): track 0.00 -> 25.8 mm
- net scaleCLK: track 51.9 -> 26.3 mm
- net PullupsBuzzer: track 0.00 -> 25.2 mm
- net Net-(A1-Pad9): track 0.00 -> 25.1 mm
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Other:
- outline, holes or cut-outs redrawn
- net class Default: via_dia 1.1 -> 2

Commit message: BOM
Parts:
- removed the REF** at (99.3, 93.3)
- removed the REF** at (95.9, 93.1)
- removed the REF** at (131.5, 49.5)
- added REF**: R_Axial_DIN0207_L6.3mm_D2.5mm_P15.24mm_Horizontal, Resistor_THT:R_Axial_DIN0207_L6.3mm_D2.5mm_P15.24mm_Horizontal, F.Cu at (146.7, 49.5)
- added REF**: R_Axial_DIN0207_L6.3mm_D2.5mm_P15.24mm_Horizontal, Resistor_THT:R_Axial_DIN0207_L6.3mm_D2.5mm_P15.24mm_Horizontal, F.Cu at (99.3, 93.2)
- added REF**: R_Axial_DIN0207_L6.3mm_D2.5mm_P15.24mm_Horizontal, Resistor_THT:R_Axial_DIN0207_L6.3mm_D2.5mm_P15.24mm_Horizontal, F.Cu at (95.9, 93.3)
- moved C3 4.91 mm to (150.4, 92.6), turned to 180 degrees
- moved C6 0.75 mm to (90.2, 94.9)
Connections:
- A1 pad 19: Net-(A1-Pad19) -> GND
- A1 pad 20: Net-(A1-Pad20) -> GND
Routing:
- net GND: track 31.1 -> 80.3 mm
- net +5V: track 211.3 -> 233.5 mm
- net scannerDATA: track 50.3 -> 51.5 mm
- net scannerCLK: track 59.9 -> 59.2 mm

Commit message: Fixed bugs
Parts:
- removed REF** (x3): R_Axial_DIN0207_L6.3mm_D2.5mm_P15.24mm_Horizontal, Resistor_THT:R_Axial_DIN0207_L6.3mm_D2.5mm_P15.24mm_Horizontal
- moved Q2 1.16 mm to (119.2, 66.7), turned to 90 degrees
- moved Q8 0.40 mm to (96.7, 66.3), turned to 90 degrees
- moved Q6 0.23 mm to (102.2, 66.3), turned to 90 degrees
- turned Q3 to 90 degrees
- turned Q5 to 90 degrees
Connections:
- Q2 pad 2: Net-(Q2-Pad2) -> GND
- Q2 pad 3: GND -> Net-(Q2-Pad3)
- Q3 pad 2: Net-(Q3-Pad2) -> GND
- Q3 pad 3: GND -> Net-(Q3-Pad3)
- Q5 pad 2: Net-(Q5-Pad2) -> GND
- Q5 pad 3: GND -> Net-(Q5-Pad3)
- Q6 pad 2: Net-(Q6-Pad2) -> GND
- Q6 pad 3: GND -> Net-(Q6-Pad3)
- Q8 pad 2: Net-(Q8-Pad2) -> GND
- Q8 pad 3: GND -> Net-(Q8-Pad3)
- R1 pad 2: Net-(Q2-Pad2) -> Net-(Q2-Pad3)
- R2 pad 2: Net-(Q3-Pad2) -> Net-(Q3-Pad3)
- R3 pad 2: Net-(Q5-Pad2) -> Net-(Q5-Pad3)
- R4 pad 2: Net-(Q6-Pad2) -> Net-(Q6-Pad3)
- R5 pad 2: Net-(Q8-Pad2) -> Net-(Q8-Pad3)
- RN1 pad 1: +5V -> GND
- RN1 pad 2: BTN -> ENCA
- RN1 pad 4: ENCA -> BTN
- enc1 pad 1: BTN -> ENCA
- enc1 pad 3: ENCA -> BTN
- enc1 pad 4: GND -> Net-(enc1-Pad4)
- enc1 pad 5: GND -> +5V
Routing:
- net +5V: track 233.5 -> 0.00 mm
- net +24V: track 159.2 -> 0.00 mm
- net GND: track 80.3 -> 0.00 mm
- net scannerCLK: track 59.2 -> 0.00 mm
- net scannerDATA: track 51.5 -> 0.00 mm
- net SCL: track 47.4 -> 0.00 mm
- net SDA: track 43.9 -> 0.00 mm
- net Buzzer: track 32.3 -> 0.00 mm
- net BTN: track 29.7 -> 0.00 mm
- net Net-(Q2-Pad2): track 29.2 -> 0.00 mm
- net ENCB: track 28.6 -> 0.00 mm
- net ENCA: track 27.3 -> 0.00 mm
- net scaleCLK: track 26.3 -> 0.00 mm
- net Net-(Q3-Pad2): track 25.8 -> 0.00 mm
- net PullupsBuzzer: track 25.2 -> 0.00 mm
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
Commit message: new layout
Parts:
- removed H1, H3, H4: MountingHole, MountingHole:MountingHole_3.2mm_M3_DIN965
- added H2: MountingHole, MountingHole:MountingHole_3.2mm_M3_DIN965, F.Cu at (170.4, 95.8)
- added H2: MountingHole, MountingHole:MountingHole_3.2mm_M3_DIN965, F.Cu at (85.4, 95.8)
- added H2: MountingHole, MountingHole:MountingHole_3.2mm_M3_DIN965, F.Cu at (170.4, 40.8)
- added JP1: Jumper, Resistor_THT:R_Axial_Power_L20.0mm_W6.4mm_P25.40mm, F.Cu at (104.7, 71.3)
- added JP2: Jumper, Resistor_THT:R_Axial_Power_L20.0mm_W6.4mm_P25.40mm, F.Cu at (154.1, 72.3)
- J1: value Barrel_Jack -> 19-24V; footprint Connector_BarrelJack:BarrelJack_Horizontal -> TerminalBlock:TerminalBlock_bornier-2_P5.08mm
- J4: value ToScanner -> Barcode scanner
- Q1, Q4, Q7: footprint Package_SO:SO-8_5.3x6.2mm_P1.27mm -> Package_SO:SOIC-8_3.9x4.9mm_P1.27mm
- Q2, Q3, Q5, Q6, Q8: footprint Package_TO_SOT_SMD:SOT-23 -> Package_TO_SOT_SMD:SOT-23_Handsoldering
- moved H2 84.5 mm to (85.4, 40.8)
- moved R6 53.9 mm to (135.5, 97.7), turned to 90 degrees
- moved R7 51.1 mm to (133.0, 97.7), turned to 90 degrees
- moved C3 22.3 mm to (166.0, 76.7), turned to 90 degrees
- moved RN2 18.3 mm to (100.9, 54.3)
- moved R1 18.2 mm to (105.3, 56.7)
- moved R2 18.2 mm to (105.3, 59.3)
- moved R3 18.2 mm to (105.3, 62.0)
- moved R4 18.2 mm to (105.3, 64.6)
- moved Q2 16.6 mm to (111.2, 52.2), turned to 180 degrees
- moved D1 16.1 mm to (152.6, 86.4), turned to 180 degrees
- moved Q8 14.5 mm to (111.2, 67.6), turned to 180 degrees
- moved R5 13.7 mm to (105.4, 67.3), turned to 0 degrees
- moved RN3 12.9 mm to (112.2, 71.9)
- moved Q4 12.5 mm to (92.2, 61.5)
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Connections:
- A1 pad 16: Buzzer -> Net-(A1-Pad16)
- J1 pad 1: Net-(F1-Pad1) -> GND
- J1 pad 2: GND -> Net-(F1-Pad1)
- J4 pad 0: Net-(J4-Pad0) -> GND
Routing:
- net +5V: track 0.00 -> 203.0 mm
- net +24V: track 0.00 -> 189.3 mm
- net scannerCLK: track 0.00 -> 54.3 mm
- net SCL: track 0.00 -> 49.7 mm
- net SDA: track 0.00 -> 49.4 mm
- net Net-(A1-Pad9): track 0.00 -> 45.7 mm
- net scannerDATA: track 0.00 -> 43.8 mm
- net Net-(A1-Pad10): track 0.00 -> 39.0 mm
- net Net-(A1-Pad11): track 0.00 -> 34.7 mm
- net L1: track 0.00 -> 33.9 mm
- net L2: track 0.00 -> 28.8 mm
- net scaleCLK: track 0.00 -> 24.4 mm
- net L3: track 0.00 -> 23.9 mm
- net Buzzer: track 0.00 -> 22.0 mm
- net scaleDATA: track 0.00 -> 20.9 mm
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