File: HW/V1/Board/Board.sch (KiCad schematic (older format))
At the start: 23 parts, among them J1 Barrel_Jack, J2 Lamp outputs, J4 ToScanner, J5 i2cLCD, J6 toScale, Q1 Si4435, Q2 Si4435, Q3 Si4435, U1 V7805-1000, U2 74HC14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

Commit message: Starting on the board
Parts:
- removed Q1, Q2, Q3: Si4435, Housings_SOIC:SOIC-8_3.9x4.9mm_Pitch1.27mm, symbol Peters:Si4435
- added J3: Lamp outputs, TerminalBlock:TerminalBlock_bornier-4_P5.08mm, symbol Connector_Generic:Conn_01x04
- added Q1, Q4, Q7: IRF7306TRPBF, Package_SO:SO-8_5.3x6.2mm_P1.27mm, symbol Peters:IRF7306TRPBF
- added Q2, Q3, Q5, Q6, Q8: BSS138, digikey-footprints:SOT-23-3, symbol dk_Transistors-FETs-MOSFETs-Single:BSS138
- added RN3: R_Network05, Resistor_THT:R_Array_SIP6, symbol Device:R_Network05
Connections:
- net labels added: Buzzer, L4, PullDownsBuzzer, PullDownsL1, PullDownsL2, PullDownsL3, PullDownsL4, PullupsBuzzer, PullupsL1, PullupsL2, PullupsL3, PullupsL4
- wire segments 38 -> 73
Other:
- moved on the sheet: A1, C2, C4, J2, RN2, U2A, U2B, U2C, U2G

Commit message: Done
Parts:
- removed J2, J3: Lamp outputs, TerminalBlock:TerminalBlock_bornier-4_P5.08mm, symbol Connector_Generic:Conn_01x04
- removed Q2, Q3, Q5, Q6, Q8: BSS138, digikey-footprints:SOT-23-3, symbol dk_Transistors-FETs-MOSFETs-Single:BSS138
- removed ROT1: ROTARY-ENCODER-Ebay, Libs:ROTARY-ENCODER-Ebay, symbol Peters:ROTARY-ENCODER-Ebay
- added D1: D_Schottky, Diode_SMD:D_SMB_Handsoldering, symbol Device:D_Schottky
- added H1, H2, H3, H4: MountingHole, MountingHole:MountingHole_3.2mm_M3_DIN965, symbol Mechanical:MountingHole
- added J2: Screw_Terminal_01x04, TerminalBlock:TerminalBlock_bornier-4_P5.08mm, symbol Connector:Screw_Terminal_01x04
- added J3: Screw_Terminal_01x02, TerminalBlock:TerminalBlock_bornier-2_P5.08mm, symbol Connector:Screw_Terminal_01x02
- added Q2, Q3, Q5, Q6, Q8: BSS138, Package_TO_SOT_SMD:SOT-23, symbol Transistor_FET:BSS138
- added R1, R2, R3, R4, R5, R6, R7: 10K, Resistor_SMD:R_0805_2012Metric_Pad1.15x1.40mm_HandSolder, symbol Device:R_Small
- added enc1: Rot_enc, Connector_PinSocket_2.54mm:PinSocket_1x05_P2.54mm_Vertical, symbol Connector:Conn_01x05_Male
- J5: footprint TerminalBlock:TerminalBlock_bornier-4_P5.08mm -> Connector_PinSocket_2.54mm:PinSocket_1x04_P2.54mm_Vertical
- Q1, Q4, Q7: symbol Peters:IRF7306TRPBF -> Board-rescue:IRF7306TRPBF-Peters
- U1: symbol dk_DC-DC-Converters:V7805-1000 -> Board-rescue:V7805-1000-dk_DC-DC-Converters
- U3: symbol Peters:HX711_Module -> Board-rescue:HX711_Module-Peters
Connections:
- wire segments 73 -> 81

Commit message: BOM
Connections:
- net GND: now also A1.19 (A0), A1.20 (A1)
Changed lines of the file:
@@
 	-1   0    0    1
 $EndComp
+$Comp
+L power:GND #PWR?
+U 1 1 5BFED80C
+P 6400 3350
+F 0 "#PWR?" H 6400 3100 50  0001 C CNN
+F 1 "GND" H 6405 3177 50  0000 C CNN
+F 2 "" H 6400 3350 50  0001 C CNN
+F 3 "" H 6400 3350 50  0001 C CNN
+	1    6400 3350
+	0    -1   -1   0
+$EndComp
+$Comp
+L power:GND #PWR?
+U 1 1 5BFED902
+P 6400 3450
+F 0 "#PWR?" H 6400 3200 50  0001 C CNN
+F 1 "GND" H 6405 3277 50  0000 C CNN
+F 2 "" H 6400 3450 50  0001 C CNN
+F 3 "" H 6400 3450 50  0001 C CNN
+	1    6400 3450
+	0    -1   -1   0
+$EndComp
 $EndSCHEMATC

Commit message: Fixed bugs
Connections:
- net +5V: now also enc1.5 (Pin_5); no longer RN1.1 (common)
- net BTN: now also RN1.4 (R3), enc1.3 (Pin_3); no longer RN1.2 (R1), enc1.1 (Pin_1)
- net ENCA: now also RN1.2 (R1), enc1.1 (Pin_1); no longer RN1.4 (R3), enc1.3 (Pin_3)
- net GND: now also Q2.2 (S), Q3.2 (S), Q5.2 (S), Q6.2 (S), Q8.2 (S), RN1.1 (common); no longer Q2.3 (D), Q3.3 (D), Q5.3 (D), Q6.3 (D), Q8.3 (D), enc1.4 (Pin_4), enc1.5 (Pin_5)
- net at R1.2: now also Q2.3 (D); no longer Q2.2 (S)
- net at R2.2: now also Q3.3 (D); no longer Q3.2 (S)
- net at R3.2: now also Q5.3 (D); no longer Q5.2 (S)
- net at R4.2: now also Q6.3 (D); no longer Q6.2 (S)
- net at R5.2: now also Q8.3 (D); no longer Q8.2 (S)
Other:
- moved on the sheet: RN1, enc1
Changed lines of the file:
@@
 L power:+5V #PWR0120
 U 1 1 5BF1D8E1
-P 5000 750
-F 0 "#PWR0120" H 5000 600 50  0001 C CNN
-F 1 "+5V" H 5015 923 50  0000 C CNN
-F 2 "" H 5000 750 50  0001 C CNN
-F 3 "" H 5000 750 50  0001 C CNN
-	1    5000 750
-	1    0    0    -1
-$EndComp
-Text GLabel 8000 900  2    50   Input ~ 0
+P 5300 700
+F 0 "#PWR0120" H 5300 550 50  0001 C CNN
+F 1 "+5V" H 5315 873 50  0000 C CNN
+F 2 "" H 5300 700 50  0001 C CNN
+F 3 "" H 5300 700 50  0001 C CNN
+	1    5300 700
+	-1   0    0    -1
+$EndComp
+Text GLabel 6000 900  2    50   Input ~ 0
 BTN
 $Comp
 L Device:R_Network05 RN1
 U 1 1 5BF1F93C
-P 5200 950
-F 0 "RN1" H 5480 996 50  0000 L CNN
-F 1 "R_Network05" H 5480 905 50  0000 L CNN
-F 2 "Resistor_THT:R_Array_SIP6" V 5575 950 50  0001 C CNN
-F 3 "http://www.vishay.com/docs/31509/csc.pdf" H 5200 950 50  0001 C CNN
-	1    5200 950
-	1    0    0    -1
-$EndComp
-$Comp
-L power:GND #PWR0122
-U 1 1 5BF209E0
-P 8000 1200
-F 0 "#PWR0122" H 8000 950 50  0001 C CNN
-F 1 "GND" H 8000 1050 50  0000 C CNN
-F 2 "" H 8000 1200 50  0001 C CNN
-F 3 "" H 8000 1200 50  0001 C CNN
-	1    8000 1200
-	0    -1   -1   0
-$EndComp
-Text GLabel 8000 1100 2    50   Input ~ 0
+P 5700 1400
+F 0 "RN1" H 5980 1446 50  0000 L CNN
+F 1 "R_Network05" H 5650 1600 50  0000 L CNN
+F 2 "Resistor_THT:R_Array_SIP6" V 6075 1400 50  0001 C CNN
+F 3 "http://www.vishay.com/docs/31509/csc.pdf" H 5700 1400 50  0001 C CNN
+	1    5700 1400
+	-1   0    0    1
+$EndComp
+Text GLabel 6000 1100 2    50   Input ~ 0
 ENCA
-Text GLabel 8000 1000 2    50   Input ~ 0
+Text GLabel 6000 1000 2    50   Input ~ 0
 ENCB
 Text GLabel 3950 3450 0    50   Input ~ 0
@@
 Text GLabel 3950 4050 0    50   Input ~ 0
 ENCA
-Text GLabel 5200 1150 3    50   Input ~ 0
-ENCA
-Text GLabel 5100 1150 3    50   Input ~ 0
-ENCB
-Text GLabel 5000 1150 3    50   Input ~ 0
-BTN
 $Comp
 L 74xx:74HC14 U2
@@
 F 3 "https://www.fairchildsemi.com/datasheets/BS/BSS138.pdf" H 1800 5750 50  0001 L CNN
 	1    1800 5750
-	-1   0    0    1
+	-1   0    0    -1
 $EndComp
 Wire Wire Line
@@
 F 3 "https://www.fairchildsemi.com/datasheets/BS/BSS138.pdf" H 3000 5900 50  0001 L CNN
 	1    3000 5900
-	-1   0    0    1
+	-1   0    0    -1
 $EndComp
 Connection ~ 3200 5900
@@
 F 3 "https://www.fairchildsemi.com/datasheets/BS/BSS138.pdf" H 4150 6000 50  0001 L CNN
 	1    4150 6000
-	-1   0    0    1
+	-1   0    0    -1
 $EndComp
 Connection ~ 4350 6000
@@
 F 3 "https://www.fairchildsemi.com/datasheets/BS/BSS138.pdf" H 5250 5900 50  0001 L CNN
 	1    5250 5900
-	-1   0    0    1
+	-1   0    0    -1
 $EndComp
 $Comp
@@
 F 3 "https://www.fairchildsemi.com/datasheets/BS/BSS138.pdf" H 6600 6050 50  0001 L CNN
 	1    6600 6050
-	-1   0    0    1
+	-1   0    0    -1
 $EndComp
 $Comp
@@
 L Connector:Conn_01x05_Male enc1
 U 1 1 5C01B864
-P 7800 1100
-F 0 "enc1" H 7906 1478 50  0000 C CNN
-F 1 "Rot_enc" H 7906 1387 50  0000 C CNN
-F 2 "Connector_PinSocket_2.54mm:PinSocket_1x05_P2.54mm_Vertical" H 7800 1100 50  0001 C CNN
-F 3 "~" H 7800 1100 50  0001 C CNN
-	1    7800 1100
-	1    0    0    -1
-$EndComp
-$Comp
-L power:GND #PWR0121
-U 1 1 5C01DE92
-P 8000 1300
-F 0 "#PWR0121" H 8000 1050 50  0001 C CNN
-F 1 "GND" H 8000 1150 50  0000 C CNN
-F 2 "" H 8000 1300 50  0001 C CNN
-F 3 "" H 8000 1300 50  0001 C CNN
-	1    8000 1300
-	0    -1   -1   0
+P 5100 900
+F 0 "enc1" V 4900 1000 50  0000 C CNN
+F 1 "Rot_enc" V 5000 950 50  0000 C CNN
+F 2 "Connector_PinSocket_2.54mm:PinSocket_1x05_P2.54mm_Vertical" H 5100 900 50  0001 C CNN
+F 3 "~" H 5100 900 50  0001 C CNN
+	1    5100 900
+	1    0    0    1
 $EndComp
 $Comp
@@
 $EndComp
 $Comp
-L power:GND #PWR?
+L power:GND #PWR0121
 U 1 1 5BFED80C
 P 6400 3350
-F 0 "#PWR?" H 6400 3100 50  0001 C CNN
+F 0 "#PWR0121" H 6400 3100 50  0001 C CNN
 F 1 "GND" H 6405 3177 50  0000 C CNN
 F 2 "" H 6400 3350 50  0001 C CNN
@@
 $EndComp
 $Comp
-L power:GND #PWR?
+L power:GND #PWR0147
 U 1 1 5BFED902
 P 6400 3450
-F 0 "#PWR?" H 6400 3200 50  0001 C CNN
+F 0 "#PWR0147" H 6400 3200 50  0001 C CNN
 F 1 "GND" H 6405 3277 50  0000 C CNN
 F 2 "" H 6400 3450 50  0001 C CNN
@@
 	0    -1   -1   0
 $EndComp
+$Comp
+L power:GND #PWR0122
+U 1 1 5BF209E0
+P 5900 1600
+F 0 "#PWR0122" H 5900 1350 50  0001 C CNN
+F 1 "GND" H 5900 1450 50  0000 C CNN
+F 2 "" H 5900 1600 50  0001 C CNN
+F 3 "" H 5900 1600 50  0001 C CNN
+	1    5900 1600
+	1    0    0    -1
+$EndComp
+Wire Wire Line
+	5300 900  5700 900
+Wire Wire Line
+	5300 1000 5800 1000
+Wire Wire Line
+	5300 1100 5900 1100
+Wire Wire Line
+	5900 1200 5900 1100
+Connection ~ 5900 1100
+Wire Wire Line
+	5900 1100 6000 1100
+Wire Wire Line
+	5800 1200 5800 1000
+Connection ~ 5800 1000
+Wire Wire Line
+	5800 1000 6000 1000
+Wire Wire Line
+	5700 1200 5700 900
+Connection ~ 5700 900
+Wire Wire Line
+	5700 900  6000 900
 $EndSCHEMATC

Commit message: new layout
Parts:
- removed J1: Barrel_Jack, Connector_BarrelJack:BarrelJack_Horizontal, symbol Connector:Barrel_Jack
- removed J4: ToScanner, Connector_Dsub:DSUB-9_Female_Horizontal_P2.77x2.84mm_EdgePinOffset7.70mm_Housed_MountingHolesOffset9.12mm, symbol Connector:DB9_Male_MountingHoles
- added J1: 19-24V, TerminalBlock:TerminalBlock_bornier-2_P5.08mm, symbol Connector:Screw_Terminal_01x02
- added J4: Barcode scanner, Connector_Dsub:DSUB-9_Female_Horizontal_P2.77x2.84mm_EdgePinOffset7.70mm_Housed_MountingHolesOffset9.12mm, symbol Connector:DB9_Female_MountingHoles
- added JP1, JP2: Jumper, Resistor_THT:R_Axial_Power_L20.0mm_W6.4mm_P25.40mm, symbol Device:Jumper
- Q1, Q4, Q7: footprint Package_SO:SO-8_5.3x6.2mm_P1.27mm -> Package_SO:SOIC-8_3.9x4.9mm_P1.27mm
- Q2, Q3, Q5, Q6, Q8: footprint Package_TO_SOT_SMD:SOT-23 -> Package_TO_SOT_SMD:SOT-23_Handsoldering
Connections:
- net +5V: now also J4.3, JP2.1, JP2.2
- net Buzzer: now also JP1.1; no longer A1.16 (D13)
- net GND: now also J1.1 (Pin_1), J4.0 (PAD), J4.1
- net scannerCLK: now also J4.7
- net scannerDATA: now also J4.9
- net at F1.1: now also J1.2 (Pin_2)
- new net: A1.16 (D13), JP1.2
Changed lines of the file:
@@
-$EndComp
-$Comp
-L Connector:Barrel_Jack J1
-U 1 1 5BF175EA
-P 1650 1600
-F 0 "J1" H 1705 1925 50  0000 C CNN
-F 1 "Barrel_Jack" H 1705 1834 50  0000 C CNN
-F 2 "Connector_BarrelJack:BarrelJack_Horizontal" H 1700 1560 50  0001 C CNN
-F 3 "~" H 1700 1560 50  0001 C CNN
-	1    1650 1600
-	1    0    0    -1
 $EndComp
 $Comp
@@
 L power:GND #PWR0102
 U 1 1 5BF19330
-P 2000 1850
-F 0 "#PWR0102" H 2000 1600 50  0001 C CNN
-F 1 "GND" H 2005 1677 50  0000 C CNN
-F 2 "" H 2000 1850 50  0001 C CNN
-F 3 "" H 2000 1850 50  0001 C CNN
-	1    2000 1850
+P 2000 1750
+F 0 "#PWR0102" H 2000 1500 50  0001 C CNN
+F 1 "GND" H 2005 1577 50  0000 C CNN
+F 2 "" H 2000 1750 50  0001 C CNN
+F 3 "" H 2000 1750 50  0001 C CNN
+	1    2000 1750
 	1    0    0    -1
 $EndComp
@@
 $EndComp
 Wire Wire Line
-	2000 1700 2000 1850
+	2000 1600 2000 1750
 Wire Wire Line
 	2400 1500 2750 1500
@@
 	0    -1   -1   0
 $EndComp
-$Comp
-L power:GND #PWR0108
-U 1 1 5BF19BED
-P 9350 3250
-F 0 "#PWR0108" H 9350 3000 50  0001 C CNN
-F 1 "GND" H 9355 3077 50  0000 C CNN
-F 2 "" H 9350 3250 50  0001 C CNN
-F 3 "" H 9350 3250 50  0001 C CNN
-	1    9350 3250
-	1    0    0    -1
-$EndComp
-Wire Wire Line
-	9400 3200 9350 3200
-Wire Wire Line
-	9350 3200 9350 3250
 Wire Wire Line
 	9400 2800 9100 2800
@@
 L power:+5V #PWR0116
 U 1 1 5BF1B326
-P 9050 4950
-F 0 "#PWR0116" H 9050 4800 50  0001 C CNN
-F 1 "+5V" H 9065 5123 50  0000 C CNN
-F 2 "" H 9050 4950 50  0001 C CNN
-F 3 "" H 9050 4950 50  0001 C CNN
-	1    9050 4950
-	-1   0    0    1
+P 8200 6050
+F 0 "#PWR0116" H 8200 5900 50  0001 C CNN
+F 1 "+5V" H 8200 6200 50  0000 C CNN
+F 2 "" H 8200 6050 50  0001 C CNN
+F 3 "" H 8200 6050 50  0001 C CNN
+	1    8200 6050
+	1    0    0    -1
 $EndComp
 $Comp
@@
 	1    0    0    -1
 $EndComp
-Text GLabel 9400 2900 0    50   Input ~ 0
+Text GLabel 9400 2700 0    50   Input ~ 0
 scannerCLK
-Text GLabel 9400 2500 0    50   Input ~ 0
+Text GLabel 9400 3100 0    50   Input ~ 0
 scannerDATA
 Text GLabel 5300 3050 0    50   Input ~ 0
@@
 P 2150 1500
 F 0 "F1" H 2150 1685 50  0000 C CNN
-F 1 "30V/1100mA" H 2200 1400 50  0000 C CNN
+F 1 "30V/1100mA" H 2150 1800 50  0000 C CNN
 F 2 "Fuse:Fuse_2920_7451Metric_Pad2.10x5.45mm_HandSolder" H 2150 1500 50  0001 C CNN
 F 3 "~" H 2150 1500 50  0001 C CNN
@@
 $EndComp
 Wire Wire Line
-	1950 1700 2000 1700
+	1950 1600 2000 1600
 Wire Wire Line
 	1950 1500 2050 1500
-$Comp
-L Connector:DB9_Male_MountingHoles J4
-U 1 1 5BF3F8D9
-P 9700 2800
-F 0 "J4" H 9880 2803 50  0000 L CNN
-F 1 "ToScanner" H 9880 2712 50  0000 L CNN
-F 2 "Connector_Dsub:DSUB-9_Female_Horizontal_P2.77x2.84mm_EdgePinOffset7.70mm_Housed_MountingHolesOffset9.12mm" H 9700 2800 50  0001 C CNN
-F 3 " ~" H 9700 2800 50  0001 C CNN
-	1    9700 2800
-	1    0    0    -1
-$EndComp
 Text GLabel 5400 3850 0    50   Input ~ 0
 L3
@@
 F 0 "Q1" H 1556 5054 50  0000 L CNN
 F 1 "IRF7306TRPBF" V 1600 5200 50  0000 L CNN
-F 2 "Package_SO:SO-8_5.3x6.2mm_P1.27mm" H 1850 5050 50  0001 C CNN
+F 2 "Package_SO:SOIC-8_3.9x4.9mm_P1.27mm" H 1850 5050 50  0001 C CNN
 F 3 "http://192.168.0.101/api/part_attachments/1126/getFile" H 1950 5150 50  0001 C CNN
 	1    1350 5100
@@
 Text GLabel 5400 3950 0    50   Input ~ 0
 L4
-Text GLabel 5400 4050 0    50   Input ~ 0
+Text GLabel 4500 4400 0    50   Input ~ 0
 Buzzer
 $Comp
@@
 F 0 "Q1" H 2756 5204 50  0000 L CNN
 F 1 "IRF7306TRPBF" V 2800 5350 50  0000 L CNN
-F 2 "Package_SO:SO-8_5.3x6.2mm_P1.27mm" H 3050 5200 50  0001 C CNN
+F 2 "Package_SO:SOIC-8_3.9x4.9mm_P1.27mm" H 3050 5200 50  0001 C CNN
 F 3 "http://192.168.0.101/api/part_attachments/1126/getFile" H 3150 5300 50  0001 C CNN
 	2    2550 5250
@@
 F 0 "Q4" H 3906 5204 50  0000 L CNN
 F 1 "IRF7306TRPBF" V 3906 5295 50  0000 L CNN
-F 2 "Package_SO:SO-8_5.3x6.2mm_P1.27mm" H 4200 5200 50  0001 C CNN
+F 2 "Package_SO:SOIC-8_3.9x4.9mm_P1.27mm" H 4200 5200 50  0001 C CNN
 F 3 "http://192.168.0.101/api/part_attachments/1126/getFile" H 4300 5300 50  0001 C CNN
 	1    3700 5250
@@
 F 0 "Q4" H 5006 5154 50  0000 L CNN
 F 1 "IRF7306TRPBF" V 5006 5245 50  0000 L CNN
-F 2 "Package_SO:SO-8_5.3x6.2mm_P1.27mm" H 5300 5150 50  0001 C CNN
+F 2 "Package_SO:SOIC-8_3.9x4.9mm_P1.27mm" H 5300 5150 50  0001 C CNN
 F 3 "http://192.168.0.101/api/part_attachments/1126/getFile" H 5400 5250 50  0001 C CNN
 	2    4800 5200
@@
 F 0 "Q7" H 6356 5404 50  0000 L CNN
 F 1 "IRF7306TRPBF" V 6356 5495 50  0000 L CNN
-F 2 "Package_SO:SO-8_5.3x6.2mm_P1.27mm" H 6650 5400 50  0001 C CNN
+F 2 "Package_SO:SOIC-8_3.9x4.9mm_P1.27mm" H 6650 5400 50  0001 C CNN
 F 3 "http://192.168.0.101/api/part_attachments/1126/getFile" H 6750 5500 50  0001 C CNN
 	1    6150 5450
@@
 F 0 "Q2" H 2006 5704 50  0000 L CNN
 F 1 "BSS138" H 2006 5795 50  0000 L CNN
-F 2 "Package_TO_SOT_SMD:SOT-23" H 2000 5675 50  0001 L CIN
+F 2 "Package_TO_SOT_SMD:SOT-23_Handsoldering" H 2000 5675 50  0001 L CIN
 F 3 "https://www.fairchildsemi.com/datasheets/BS/BSS138.pdf" H 1800 5750 50  0001 L CNN
 	1    1800 5750
@@
 F 0 "Q3" H 3206 5854 50  0000 L CNN
 F 1 "BSS138" H 3206 5945 50  0000 L CNN
-F 2 "Package_TO_SOT_SMD:SOT-23" H 3200 5825 50  0001 L CIN
+F 2 "Package_TO_SOT_SMD:SOT-23_Handsoldering" H 3200 5825 50  0001 L CIN
 F 3 "https://www.fairchildsemi.com/datasheets/BS/BSS138.pdf" H 3000 5900 50  0001 L CNN
 	1    3000 5900
@@
 F 0 "Q5" H 4356 5954 50  0000 L CNN
 F 1 "BSS138" H 4356 6045 50  0000 L CNN
-F 2 "Package_TO_SOT_SMD:SOT-23" H 4350 5925 50  0001 L CIN
+F 2 "Package_TO_SOT_SMD:SOT-23_Handsoldering" H 4350 5925 50  0001 L CIN
 F 3 "https://www.fairchildsemi.com/datasheets/BS/BSS138.pdf" H 4150 6000 50  0001 L CNN
 	1    4150 6000
@@
 F 0 "Q6" H 5456 5854 50  0000 L CNN
 F 1 "BSS138" H 5456 5945 50  0000 L CNN
-F 2 "Package_TO_SOT_SMD:SOT-23" H 5450 5825 50  0001 L CIN
+F 2 "Package_TO_SOT_SMD:SOT-23_Handsoldering" H 5450 5825 50  0001 L CIN
 F 3 "https://www.fairchildsemi.com/datasheets/BS/BSS138.pdf" H 5250 5900 50  0001 L CNN
 	1    5250 5900
@@
 F 0 "Q8" H 6806 6004 50  0000 L CNN
 F 1 "BSS138" H 6806 6095 50  0000 L CNN
-F 2 "Package_TO_SOT_SMD:SOT-23" H 6800 5975 50  0001 L CIN
+F 2 "Package_TO_SOT_SMD:SOT-23_Handsoldering" H 6800 5975 50  0001 L CIN
 F 3 "https://www.fairchildsemi.com/datasheets/BS/BSS138.pdf" H 6600 6050 50  0001 L CNN
 	1    6600 6050
@@
 Wire Wire Line
 	5700 900  6000 900
+$Comp
+L Connector:DB9_Female_MountingHoles J4
+U 1 1 5C004D8E
+P 9700 2800
+F 0 "J4" H 9880 2803 50  0000 L CNN
+F 1 "Barcode scanner" V 10000 2300 50  0000 L CNN
+F 2 "Connector_Dsub:DSUB-9_Female_Horizontal_P2.77x2.84mm_EdgePinOffset7.70mm_Housed_MountingHolesOffset9.12mm" H 9700 2800 50  0001 C CNN
+F 3 " ~" H 9700 2800 50  0001 C CNN
+	1    9700 2800
+	1    0    0    -1
+$EndComp
+$Comp
+L power:GND #PWR0148
+U 1 1 5C0054AD
+P 9700 3400
+F 0 "#PWR0148" H 9700 3150 50  0001 C CNN
+F 1 "GND" H 9705 3227 50  0000 C CNN
+F 2 "" H 9700 3400 50  0001 C CNN
+F 3 "" H 9700 3400 50  0001 C CNN
+	1    9700 3400
+	1    0    0    -1
+$EndComp
+$Comp
+L power:GND #PWR0108
+U 1 1 5C0069B4
+P 9400 2400
+F 0 "#PWR0108" H 9400 2150 50  0001 C CNN
+F 1 "GND" H 9405 2227 50  0000 C CNN
+F 2 "" H 9400 2400 50  0001 C CNN
+F 3 "" H 9400 2400 50  0001 C CNN
+	1    9400 2400
+	0    1    1    0
+$EndComp
+$Comp
+L Connector:Screw_Terminal_01x02 J1
+U 1 1 5C007403
+P 1750 1600
+F 0 "J1" H 1670 1275 50  0000 C CNN
+F 1 "19-24V" V 1900 1550 50  0000 C CNN
+F 2 "TerminalBlock:TerminalBlock_bornier-2_P5.08mm" H 1750 1600 50  0001 C CNN
+F 3 "~" H 1750 1600 50  0001 C CNN
+	1    1750 1600
+	-1   0    0    1
+$EndComp
+$Comp
+L Device:Jumper JP2
+U 1 1 5C00CA36
+P 8500 6050
+F 0 "JP2" H 8500 6314 50  0000 C CNN
+F 1 "Jumper" H 8500 6223 50  0000 C CNN
+F 2 "Resistor_THT:R_Axial_Power_L20.0mm_W6.4mm_P25.40mm" H 8500 6050 50  0001 C CNN
+F 3 "~" H 8500 6050 50  0001 C CNN
+	1    8500 6050
+	1    0    0    -1
+$EndComp
+$Comp
+L Device:Jumper JP1
+U 1 1 5C00F01F
+P 4800 4400
+F 0 "JP1" H 4800 4664 50  0000 C CNN
+F 1 "Jumper" H 4800 4573 50  0000 C CNN
+F 2 "Resistor_THT:R_Axial_Power_L20.0mm_W6.4mm_P25.40mm" H 4800 4400 50  0001 C CNN
+F 3 "~" H 4800 4400 50  0001 C CNN
+	1    4800 4400
+	1    0    0    -1
+$EndComp
+Wire Wire Line
+	5100 4400 5400 4400
+Wire Wire Line
+	5400 4400 5400 4050
+$Comp
+L power:+5V #PWR?
+U 1 1 5C012276
+P 8800 6050
+F 0 "#PWR?" H 8800 5900 50  0001 C CNN
+F 1 "+5V" H 8800 6200 50  0000 C CNN
+F 2 "" H 8800 6050 50  0001 C CNN
+F 3 "" H 8800 6050 50  0001 C CNN
+	1    8800 6050
+	1    0    0    -1
+$EndComp
+$Comp
+L power:+5V #PWR?
+U 1 1 5C0122E3
+P 8800 5150
+F 0 "#PWR?" H 8800 5000 50  0001 C CNN
+F 1 "+5V" H 8800 5300 50  0000 C CNN
+F 2 "" H 8800 5150 50  0001 C CNN
+F 3 "" H 8800 5150 50  0001 C CNN
+	1    8800 5150
+	1    0    0    -1
+$EndComp
+Wire Wire Line
+	8800 5150 9050 5150
+Wire Wire Line
+	9050 5150 9050 4950
 $EndSCHEMATC
